Commit message: add sim

File: urdf/my_robot.xacro (robot description, xacro)
@@ -4,10 +4,10 @@
         <visual>
             <geometry>
-                <box size="0.1 0.1 0.1"/>
+                <box size="0.15 0.15 0.3"/>
             </geometry>
         </visual>
         <collision>
             <geometry>
-                <box size="0.1 0.1 0.1"/>
+                <box size="0.15 0.15 0.3"/>
             </geometry>
         </collision>
@@ -41,5 +41,5 @@
         <dynamics damping="1.0" friction="0.5"/>
         <limit effort="5.0" lower="-1e9" upper="1e9" velocity="5.0"/>
-        <origin xyz="0.0 0.0 0.1" rpy="0.0 0.0 0.0"/>
+        <origin xyz="0.0 0.0 0.2" rpy="0.0 0.0 0.0"/>
     </joint>
     <transmission name="joint1_trans">
@@ -53,3 +53,9 @@
         </joint>
     </transmission>
+    <gazebo>
+        <plugin name="rm_ros_control" filename="librm_robot_hw_sim.so">
+            <robotNamespace>/</robotNamespace>
+            <robotSimType>rm_gazebo/RmRobotHWSim</robotSimType>
+        </plugin>
+    </gazebo>
 </robot>
